File: HIL Breakout Board 3.3.kicad_pcb (KiCad board)
At the start: 6 copper layers, 262.5 x 110.2 mm, 42 parts, among them J1 DIN41612_03x32_C_Split, J10 Conn_01x32_Pin, J2 DIN41612_03x32_C_Split, J3 Conn_01x32_Pin, J4 2-5174225-5, J5 2-5174225-5, J6 Conn_01x32_Pin, J7 Conn_01x32_Pin, J8 Conn_01x32_Pin, J9 Conn_01x32_Pin

Commit message: Fixed the logo placement and added SEES
Other:
- board text added: "Created by: Kevin Monahan Eric Schmitt HIL to NI Board V1.1 4/10/2026"
- board text added: "SEES"
- board text removed: "Created by: Kevin Monahan Eric Schmitt HIL to NI Board V1.1"

Commit message: Minor changes to board
Routing:
- net DO24: track 114.8 -> 112.0 mm
